File: RelayDiagram/OpenThermostat.sch (KiCad schematic (older format))
At the start: 99 parts, among them J1 Conn_01x08_Female, J2 Conn_01x15_Female, J3 Conn_01x15_Female, J4 Conn_01x09_Female, Q1 Q_NMOS_DGS, Q10 Q_NMOS_DGS, Q11 Q_NMOS_DGS, Q12 Q_NMOS_DGS, Q2 Q_NMOS_DGS, Q3 Q_NMOS_DGS, Q4 Q_NMOS_DGS, Q5 Q_NMOS_DGS, Q6 Q_NMOS_DGS, Q7 Q_NMOS_DGS, Q8 Q_NMOS_DGS, Q9 Q_NMOS_DGS, SW2 SW_Push, SW3 SW_Push, SW4 SW_Push, SW5 SW_Push, SW6 SW_Push, U1 PCF8574, U10 MB10S-13, U11 L7805CV, U2 LCD, U3 DHT11, U4 EE2-3TNU-L_DPDT_Relay, U5 EE2-3TNU-L_DPDT_Relay, U6 EE2-3TNU-L_DPDT_Relay, U7 EE2-3TNU-L_DPDT_Relay, U8 EE2-3TNU-L_DPDT_Relay, U9 EE2-3TNU-L_DPDT_Relay

Commit message: Fixed relay R & RC connections, removed 1M ohm series button resistors, added 5V and GND to I/O header
Parts:
- removed J1: Conn_01x08_Female, Pin_Headers:Pin_Header_Angled_1x03_Pitch1.27mm, symbol Connector:Conn_01x08_Female
- removed R5, R6, R7, R8, R9: 1M, Resistors_SMD:R_0805, symbol Device:R
- added J1: Conn_01x10_Female, Pin_Headers:Pin_Header_Angled_1x10_Pitch2.54mm, symbol conn:Conn_01x10_Female
- C1, C2, C3: symbol OpenThermostat-rescue:Capacitor_Unpolarized-solarcar-device-OpenThermostat-rescue-OpenThermostat-rescue -> OpenThermostat-rescue:Capacitor_Unpolarized-solarcar-device-OpenThermostat-rescue-OpenThermostat-rescue-OpenThermostat-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
- U10: symbol OpenThermostat-rescue:MB10S-13-OpenThermostat-rescue-OpenThermostat-rescue-OpenThermostat-rescue -> OpenThermostat-rescue:MB10S-13-OpenThermostat-rescue-OpenThermostat-rescue-OpenThermostat-rescue-OpenThermostat-rescue
- U11: symbol OpenThermostat-rescue:L7805CV-OpenThermostat-rescue-OpenThermostat-rescue-OpenThermostat-rescue -> OpenThermostat-rescue:L7805CV-OpenThermostat-rescue-OpenThermostat-rescue-OpenThermostat-rescue-OpenThermostat-rescue
Connections:
- wire segments 491 -> 490
Changed lines of the file:
@@
 R
-$Comp
-L Connector:Conn_01x08_Female J1
-U 1 1 5D5018A7
-P 1935 725
-F 0 "J1" V 2100 655 50  0000 C CNN
-F 1 "Conn_01x08_Female" V 2009 655 50  0000 C CNN
-F 2 "Pin_Headers:Pin_Header_Angled_1x03_Pitch1.27mm" H 1935 725 50  0001 C CNN
-F 3 "~" H 1935 725 50  0001 C CNN
-	1    1935 725
-	0    -1   -1   0
-$EndComp
 $Comp
 L SeniorDesignLibrary:EE2-3TNU-L_DPDT_Relay U8
@@
 	1    7950 7575
 	-1   0    0    -1
-$EndComp
-$Comp
-L Device:R R5
-U 1 1 5C5A6D12
-P 3760 6190
-F 0 "R5" H 3650 6330 50  0000 L CNN
-F 1 "1M" V 3760 6130 50  0000 L CNN
-F 2 "Resistors_SMD:R_0805" V 3690 6190 50  0001 C CNN
-F 3 "~" H 3760 6190 50  0001 C CNN
-	1    3760 6190
-	1    0    0    -1
-$EndComp
-$Comp
-L Device:R R6
-U 1 1 5C7E067D
-P 3880 6190
-F 0 "R6" H 3770 6330 50  0000 L CNN
-F 1 "1M" V 3880 6130 50  0000 L CNN
-F 2 "Resistors_SMD:R_0805" V 3810 6190 50  0001 C CNN
-F 3 "~" H 3880 6190 50  0001 C CNN
-	1    3880 6190
-	1    0    0    -1
-$EndComp
-$Comp
-L Device:R R7
-U 1 1 5C7E089B
-P 3990 6190
-F 0 "R7" H 3890 6330 50  0000 L CNN
-F 1 "1M" V 3990 6130 50  0000 L CNN
-F 2 "Resistors_SMD:R_0805" V 3920 6190 50  0001 C CNN
-F 3 "~" H 3990 6190 50  0001 C CNN
-	1    3990 6190
-	1    0    0    -1
-$EndComp
-$Comp
-L Device:R R8
-U 1 1 5C7E10D8
-P 4110 6190
-F 0 "R8" H 4000 6330 50  0000 L CNN
-F 1 "1M" V 4110 6130 50  0000 L CNN
-F 2 "Resistors_SMD:R_0805" V 4040 6190 50  0001 C CNN
-F 3 "~" H 4110 6190 50  0001 C CNN
-	1    4110 6190
-	1    0    0    -1
-$EndComp
-$Comp
-L Device:R R9
-U 1 1 5C7E13A6
-P 4225 6190
-F 0 "R9" H 4125 6330 50  0000 L CNN
-F 1 "1M" V 4225 6130 50  0000 L CNN
-F 2 "Resistors_SMD:R_0805" V 4155 6190 50  0001 C CNN
-F 3 "~" H 4225 6190 50  0001 C CNN
-	1    4225 6190
-	1    0    0    -1
 $EndComp
 $Comp
@@
 $EndComp
 $Comp
-L OpenThermostat-rescue:MB10S-13-OpenThermostat-rescue-OpenThermostat-rescue-OpenThermostat-rescue U10
+L OpenThermostat-rescue:MB10S-13-OpenThermostat-rescue-OpenThermostat-rescue-OpenThermostat-rescue-OpenThermostat-rescue U10
 U 1 1 5C64C7AA
 P 10975 2675
@@
 R
 $Comp
-L OpenThermostat-rescue:L7805CV-OpenThermostat-rescue-OpenThermostat-rescue-OpenThermostat-rescue U11
+L OpenThermostat-rescue:L7805CV-OpenThermostat-rescue-OpenThermostat-rescue-OpenThermostat-rescue-OpenThermostat-rescue U11
 U 1 1 5C651BD2
 P 10975 3425
@@
 $EndComp
 $Comp
-L OpenThermostat-rescue:Capacitor_Unpolarized-solarcar-device-OpenThermostat-rescue-OpenThermostat-rescue C1
+L OpenThermostat-rescue:Capacitor_Unpolarized-solarcar-device-OpenThermostat-rescue-OpenThermostat-rescue-OpenThermostat-rescue C1
 U 1 1 5C65344A
 P 11450 2675
@@
 	2750 2825 2720 2825
 Wire Wire Line
-	1095 925  1095 1670
-Wire Wire Line
 	1195 1670 1195 1050
 Wire Wire Line
@@
 	6700 9750 7550 9750
 Wire Wire Line
-	3760 6680 3760 6340
-Wire Wire Line
-	3880 6685 3880 6340
-Wire Wire Line
-	3990 6340 3990 6680
-Wire Wire Line
-	4110 6685 4110 6340
-Wire Wire Line
-	4225 6685 4225 6340
-Wire Wire Line
-	3760 4720 3760 6040
-Wire Wire Line
-	3880 4695 3880 6040
-Wire Wire Line
-	3990 4640 3990 6040
-Wire Wire Line
 	8400 8800 8425 8800
 Wire Wire Line
@@
 Wire Wire Line
 	3950 2725 4165 2725
-Wire Wire Line
-	1095 925  1635 925
 Connection ~ 8350 6200
 Connection ~ 8350 7875
@@
 $EndComp
 $Comp
-L OpenThermostat-rescue:Capacitor_Unpolarized-solarcar-device-OpenThermostat-rescue-OpenThermostat-rescue C3
+L OpenThermostat-rescue:Capacitor_Unpolarized-solarcar-device-OpenThermostat-rescue-OpenThermostat-rescue-OpenThermostat-rescue C3
 U 1 1 5C778E29
 P 3950 2575
@@
 $EndComp
 $Comp
-L OpenThermostat-rescue:Capacitor_Unpolarized-solarcar-device-OpenThermostat-rescue-OpenThermostat-rescue C2
+L OpenThermostat-rescue:Capacitor_Unpolarized-solarcar-device-OpenThermostat-rescue-OpenThermostat-rescue-OpenThermostat-rescue C2
 U 1 1 5C77A8FC
 P 1635 4740
@@
 	1655 4565 4725 4565
 Wire Wire Line
-	4110 6040 4110 4230
-Wire Wire Line
 	4110 3825 3950 3825
 Wire Wire Line
@@
 	2625 3395 2625 4405
 Connection ~ 4225 4405
-Wire Wire Line
-	4225 4405 4225 6040
 Connection ~ 2525 2725
 Wire Wire Line
 	2750 2725 2525 2725
+Wire Wire Line
+	4225 4405 4225 6685
+Wire Wire Line
+	4110 4230 4110 6685
+Wire Wire Line
+	3990 4640 3990 6680
+Wire Wire Line
+	3880 4695 3880 6685
+Wire Wire Line
+	3760 4720 3760 6680
+$Comp
+L conn:Conn_01x10_Female J1
+U 1 1 5D4716B1
+P 1835 725
+F 0 "J1" V 2000 655 50  0000 C CNN
+F 1 "Conn_01x10_Female" V 1909 655 50  0000 C CNN
+F 2 "Pin_Headers:Pin_Header_Angled_1x10_Pitch2.54mm" H 1835 725 50  0001 C CNN
+F 3 "~" H 1835 725 50  0001 C CNN
+	1    1835 725
+	0    -1   -1   0
+$EndComp
+$Comp
+L power:GND #PWR0106
+U 1 1 5D531BE3
+P 1535 925
+F 0 "#PWR0106" H 1535 675 50  0001 C CNN
+F 1 "GND" H 1540 752 50  0000 C CNN
+F 2 "" H 1535 925 50  0001 C CNN
+F 3 "" H 1535 925 50  0001 C CNN
+	1    1535 925
+	1    0    0    -1
+$EndComp
+Wire Wire Line
+	1635 925  1635 1025
+Wire Wire Line
+	1635 1025 1095 1025
+Wire Wire Line
+	1095 1025 1095 1670
+$Comp
+L power:+5V #PWR0105
+U 1 1 5D4723B8
+P 1250 920
+F 0 "#PWR0105" H 1250 770 50  0001 C CNN
+F 1 "+5V" H 1185 1095 50  0000 L CNN
+F 2 "" H 1250 920 50  0001 C CNN
+F 3 "" H 1250 920 50  0001 C CNN
+	1    1250 920
+	1    0    0    -1
+$EndComp
+Wire Wire Line
+	1250 920  1250 980
+Wire Wire Line
+	1250 980  1435 980
+Wire Wire Line
+	1435 980  1435 925
 $EndSCHEMATC
